File: spindle_driver.kicad_pcb (KiCad board)
At the start: 2 copper layers, 68 x 98 mm, 97 parts, among them J1 Hall Sensors, J10 RJ12_Shielded, J11 EXPANSION, J12 EXPANSION, J2 INLC, J3 INHB, J4 INLA, J5 Motor, J6 JTAG/SWD, J7 M_PWR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

Commit message: Updated project to Kicad 8
Other:
- net class Default removed
- net class Power removed
