File: pwr&io.kicad_sch (KiCad schematic)
At the start: 25 parts, among them J10 Field_Bus_Out, J11 EXPANSION, J12 EXPANSION, J8 USB_B, J9 Field_Bus_In, SW3 TERM_EN, U3 USBLC6-2SC6, U4 TPS54336ADDA, U5 ST1480ABDR

Commit message: Added project description
Parts:
- renumbered J8 to J?, U4 to U?
Changed lines of the file:
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@@
 		(on_board yes)
 		(dnp no)
-		(property "Reference" "U4"
+		(property "Reference" "U?"
 			(at 218.44 51.6382 0)
 			(effects
@@
 		(on_board yes)
 		(dnp no)
-		(property "Reference" "#PWR045"
+		(property "Reference" "#PWR?"
 			(at 76.2 138.43 0)
 			(effects
@@
 		(on_board yes)
 		(dnp no)
-		(property "Reference" "#PWR043"
+		(property "Reference" "#PWR?"
 			(at 62.23 127 0)
 			(effects
@@
 		(on_board yes)
 		(dnp no)
-		(property "Reference" "#PWR048"
+		(property "Reference" "#PWR?"
 			(at 62.23 163.83 0)
 			(effects
@@
 		(on_board yes)
 		(dnp no)
-		(property "Reference" "#PWR037"
+		(property "Reference" "#PWR?"
 			(at 73.66 67.31 0)
 			(effects
@@
 		(on_board yes)
 		(dnp no)
-		(property "Reference" "J8"
+		(property "Reference" "J?"
 			(at 49.7078 45.2882 0)
 			(effects
@@
 		(on_board yes)
 		(dnp no)
-		(property "Reference" "#PWR039"
+		(property "Reference" "#PWR?"
 			(at 48.26 78.74 0)
 			(effects
@@
 		(on_board yes)
 		(dnp no)
-		(property "Reference" "#PWR049"
+		(property "Reference" "#PWR?"
 			(at 49.53 134.62 0)
 			(effects
@@
 		(on_board yes)
 		(dnp no)
-		(property "Reference" "#PWR040"
+		(property "Reference" "#PWR?"
 			(at 215.9 90.17 0)
 			(effects
